Commit message: Imported upstream version '4.1.0' of 'upstream'

File: urdf/ur.urdf.xacro (robot description, xacro)
@@ -5,5 +5,5 @@
    <!-- import main macro -->
    <xacro:include filename="$(find ur_description)/urdf/ur_macro.xacro"/>
-   <!-- possible 'ur_type' values: ur3, ur3e, ur5, ur5e, ur7e, ur10, ur10e, ur12e, ur16e, ur15, ur20, ur30 -->
+   <!-- possible 'ur_type' values: ur3, ur5, ur10, ur3e, ur5e, ur7e, ur10e, ur12e, ur16e, ur8long, ur15, ur20, ur30 -->
    <!-- the default value should raise an error in case this was called without defining the type -->
    <xacro:arg name="ur_type" default="ur5x"/>

File: urdf/ur_macro.xacro (robot description, xacro)
@@ -8,5 +8,5 @@
     This file models the base kinematic chain of a UR robot, which then gets
     parameterised by various configuration files to convert it into a UR3(e),
-    UR5(e), UR10(e) or UR16e.
+    UR5(e), UR10(e) or UR16e, etc.
     NOTE the default kinematic parameters (i.e., link lengths, frame locations,
     offsets, etc) do not correspond to any particular robot. They are defaults
@@ -73,6 +73,9 @@
     <link name="${tf_prefix}base_link"/>
     <link name="${tf_prefix}base_link_inertia">
-      <visual>
-        <origin xyz="0 0 0" rpy="0 0 ${pi}"/>
+      <xacro:get_visual_params name="base" type="mesh_offset"/>
+      <visual>
+        <origin
+         xyz="${visual_params['x']} ${visual_params['y']} ${visual_params['z']}"
+         rpy="${visual_params['roll']} ${visual_params['pitch']} ${visual_params['yaw']}"/>
         <geometry>
           <xacro:get_mesh name="base" type="visual"/>
@@ -80,5 +83,7 @@
       </visual>
       <collision>
-        <origin xyz="0 0 0" rpy="0 0 ${pi}"/>
+        <origin
+         xyz="${visual_params['x']} ${visual_params['y']} ${visual_params['z']}"
+         rpy="${visual_params['roll']} ${visual_params['pitch']} ${visual_params['yaw']}"/>
         <geometry>
           <xacro:get_mesh name="base" type="collision"/>
@@ -90,6 +95,9 @@
     </link>
     <link name="${tf_prefix}shoulder_link">
-      <visual>
-        <origin xyz="0 0 0" rpy="0 0 ${pi}"/>
+      <xacro:get_visual_params name="shoulder" type="mesh_offset"/>
+      <visual>
+        <origin
+         xyz="${visual_params['x']} ${visual_params['y']} ${visual_params['z']}"
+         rpy="${visual_params['roll']} ${visual_params['pitch']} ${visual_params['yaw']}"/>
         <geometry>
           <xacro:get_mesh name="shoulder" type="visual"/>
@@ -97,5 +105,7 @@
       </visual>
       <collision>
-        <origin xyz="0 0 0" rpy="0 0 ${pi}"/>
+        <origin
+         xyz="${visual_params['x']} ${visual_params['y']} ${visual_params['z']}"
+         rpy="${visual_params['roll']} ${visual_params['pitch']} ${visual_params['yaw']}"/>
         <geometry>
           <xacro:get_mesh name="shoulder" type="collision"/>
@@ -115,6 +125,9 @@
       </inertial>    </link>
     <link name="${tf_prefix}upper_arm_link">
-      <visual>
-        <origin xyz="0 0 ${shoulder_offset}" rpy="${pi/2} 0 ${-pi/2}"/>
+      <xacro:get_visual_params name="upper_arm" type="mesh_offset"/>
+      <visual>
+        <origin
+         xyz="${visual_params['x']} ${visual_params['y']} ${visual_params['z']}"
+         rpy="${visual_params['roll']} ${visual_params['pitch']} ${visual_params['yaw']}"/>
         <geometry>
           <xacro:get_mesh name="upper_arm" type="visual"/>
@@ -122,5 +135,7 @@
       </visual>
       <collision>
-        <origin xyz="0 0 ${shoulder_offset}" rpy="${pi/2} 0 ${-pi/2}"/>
+        <origin
+         xyz="${visual_params['x']} ${visual_params['y']} ${visual_params['z']}"
+         rpy="${visual_params['roll']} ${visual_params['pitch']} ${visual_params['yaw']}"/>
         <geometry>
           <xacro:get_mesh name="upper_arm" type="collision"/>
@@ -141,6 +156,9 @@
     </link>
     <link name="${tf_prefix}forearm_link">
-      <visual>
-        <origin xyz="0 0 ${elbow_offset}" rpy="${pi/2} 0 ${-pi/2}"/>
+      <xacro:get_visual_params name="forearm" type="mesh_offset"/>
+      <visual>
+        <origin
+         xyz="${visual_params['x']} ${visual_params['y']} ${visual_params['z']}"
+         rpy="${visual_params['roll']} ${visual_params['pitch']} ${visual_params['yaw']}"/>
         <geometry>
           <xacro:get_mesh name="forearm" type="visual"/>
@@ -148,5 +166,7 @@
       </visual>
       <collision>
-        <origin xyz="0 0 ${elbow_offset}" rpy="${pi/2} 0 ${-pi/2}"/>
+        <origin
+         xyz="${visual_params['x']} ${visual_params['y']} ${visual_params['z']}"
+         rpy="${visual_params['roll']} ${visual_params['pitch']} ${visual_params['yaw']}"/>
         <geometry>
           <xacro:get_mesh name="forearm" type="collision"/>
@@ -167,7 +187,9 @@
     </link>
     <link name="${tf_prefix}wrist_1_link">
-	  <xacro:get_visual_params name="wrist_1" type="visual_offset"/>
-      <visual>
-      	<origin xyz="0 0 ${visual_params}" rpy="${pi/2} 0 0"/>
+      <xacro:get_visual_params name="wrist_1" type="mesh_offset"/>
+      <visual>
+        <origin
+         xyz="${visual_params['x']} ${visual_params['y']} ${visual_params['z']}"
+         rpy="${visual_params['roll']} ${visual_params['pitch']} ${visual_params['yaw']}"/>
         <geometry>
           <xacro:get_mesh name="wrist_1" type="visual"/>
@@ -175,5 +197,7 @@
       </visual>
       <collision>
-        <origin xyz="0 0 ${visual_params}" rpy="${pi/2} 0 0"/>
+        <origin
+         xyz="${visual_params['x']} ${visual_params['y']} ${visual_params['z']}"
+         rpy="${visual_params['roll']} ${visual_params['pitch']} ${visual_params['yaw']}"/>
         <geometry>
           <xacro:get_mesh name="wrist_1" type="collision"/>
@@ -194,7 +218,9 @@
     </link>
     <link name="${tf_prefix}wrist_2_link">
-          <xacro:get_visual_params name="wrist_2" type="visual_offset"/>
-      <visual>
-        <origin xyz="0 0 ${visual_params}" rpy="0 0 0"/>
+      <xacro:get_visual_params name="wrist_2" type="mesh_offset"/>
+      <visual>
+        <origin
+         xyz="${visual_params['x']} ${visual_params['y']} ${visual_params['z']}"
+         rpy="${visual_params['roll']} ${visual_params['pitch']} ${visual_params['yaw']}"/>
         <geometry>
           <xacro:get_mesh name="wrist_2" type="visual"/>
@@ -202,5 +228,7 @@
       </visual>
       <collision>
-        <origin xyz="0 0 ${visual_params}" rpy="0 0 0"/>
+        <origin
+         xyz="${visual_params['x']} ${visual_params['y']} ${visual_params['z']}"
+         rpy="${visual_params['roll']} ${visual_params['pitch']} ${visual_params['yaw']}"/>
         <geometry>
           <xacro:get_mesh name="wrist_2" type="collision"/>
@@ -221,13 +249,9 @@
     </link>
     <link name="${tf_prefix}wrist_3_link">
-      <!-- TODO: remove this once all wrist_3 meshes have the visual_offset_xyz tag -->
-      <xacro:get_visual_params name="wrist_3" type="visual_offset_xyz"/>
-      <xacro:property name="mesh_offset" value="${visual_params}" scope="parent"/>
-      <xacro:if value="${visual_params == ''}">
-        <xacro:get_visual_params name="wrist_3" type="visual_offset"/>
-        <xacro:property name="mesh_offset" value="0 0 ${visual_params}" scope="parent"/>
-      </xacro:if>
-      <visual>
-        <origin xyz="${mesh_offset}" rpy="${pi/2} 0 0"/>
+      <xacro:get_visual_params name="wrist_3" type="mesh_offset"/>
+      <visual>
+        <origin
+         xyz="${visual_params['x']} ${visual_params['y']} ${visual_params['z']}"
+         rpy="${visual_params['roll']} ${visual_params['pitch']} ${visual_params['yaw']}"/>
         <geometry>
           <xacro:get_mesh name="wrist_3" type="visual"/>
@@ -235,5 +259,7 @@
       </visual>
       <collision>
-        <origin xyz="${mesh_offset}" rpy="${pi/2} 0 0"/>
+        <origin
+         xyz="${visual_params['x']} ${visual_params['y']} ${visual_params['z']}"
+         rpy="${visual_params['roll']} ${visual_params['pitch']} ${visual_params['yaw']}"/>
         <geometry>
           <xacro:get_mesh name="wrist_3" type="collision"/>

File: urdf/ur_mocked.urdf.xacro (robot description, xacro)
@@ -6,5 +6,5 @@
   <xacro:include filename="$(find ur_description)/urdf/ur_macro.xacro"/>
   <xacro:include filename="$(find ur_description)/urdf/ros2_control_mock_hardware.xacro" />
-  <!-- possible 'ur_type' values: ur3, ur3e, ur5, ur5e, ur7e, ur10, ur10e, ur12e, ur16e, ur15, ur20, ur30 -->
+  <!-- possible 'ur_type' values: ur3, ur5, ur10, ur3e, ur5e, ur7e, ur10e, ur12e, ur16e, ur8long, ur15, ur20, ur30 -->
   <!-- the default value should raise an error in case this was called without defining the type -->
   <xacro:arg name="ur_type" default="ur5x"/>

Commit message: Imported upstream version '2.7.0' of 'upstream'

File: urdf/ur.urdf.xacro (robot description, xacro)
@@ -18,8 +18,63 @@
    <xacro:arg name="safety_pos_margin" default="0.15"/>
    <xacro:arg name="safety_k_position" default="20"/>
-   <!--When using gazebo simulations absolute paths are necessary.-->
-   <xacro:arg name="force_abs_paths" default="false" />
+   <!-- ros2_control related parameters -->
+   <xacro:arg name="headless_mode" default="false" />
+   <xacro:arg name="robot_ip" default="0.0.0.0" />
+   <xacro:arg name="script_filename" default=""/>
+   <xacro:arg name="output_recipe_filename" default=""/>
+   <xacro:arg name="input_recipe_filename" default=""/>
+   <xacro:arg name="reverse_ip" default="0.0.0.0"/>
+   <xacro:arg name="script_command_port" default="50004"/>
+   <xacro:arg name="reverse_port" default="50001"/>
+   <xacro:arg name="script_sender_port" default="50002"/>
+   <xacro:arg name="trajectory_port" default="50003"/>
+   <!--   tool communication related parameters-->
+   <xacro:arg name="use_tool_communication" default="false" />
+   <xacro:arg name="tool_voltage" default="0" />
+   <xacro:arg name="tool_parity" default="0" />
+   <xacro:arg name="tool_baud_rate" default="115200" />
+   <xacro:arg name="tool_stop_bits" default="1" />
+   <xacro:arg name="tool_rx_idle_chars" default="1.5" />
+   <xacro:arg name="tool_tx_idle_chars" default="3.5" />
+   <xacro:arg name="tool_device_name" default="/tmp/ttyUR" />
+   <xacro:arg name="tool_tcp_port" default="54321" />
+     <!-- Simulation parameters -->
+   <xacro:arg name="use_fake_hardware" default="false" />
+   <xacro:arg name="fake_sensor_commands" default="false" />
+   <xacro:arg name="sim_gazebo" default="false" />
+   <xacro:arg name="sim_ignition" default="false" />
+   <xacro:arg name="simulation_controllers" default="" />
+   <!-- initial position for simulations (Fake Hardware, Gazebo, Ignition) -->
+   <xacro:arg name="initial_positions_file" default="$(find ur_description)/config/initial_positions.yaml"/>
+   <!-- convert to property to use substitution in function -->
+   <xacro:property name="initial_positions_file" default="$(arg initial_positions_file)"/>
+   <xacro:property name="is_sim_gazebo" value="$(arg sim_gazebo)"/>
+   <xacro:property name="is_sim_ignition" value="$(arg sim_ignition)"/>
    <!-- create link fixed to the "world" -->
    <link name="world" />
+   <xacro:if value="${is_sim_gazebo or is_sim_ignition}">
+     <link name="ground_plane">
+       <visual>
+         <origin rpy="0 0 0" xyz="0 0 0"/>
+         <geometry>
+           <box size="5 5 0"/>
+         </geometry>
+         <material name="ground_white">
+           <color rgba="1 1 1 0.5"/>
+         </material>
+       </visual>
+       <collision>
+         <origin rpy="0 0 0" xyz="0 0 0"/>
+         <geometry>
+           <box size="5 5 0"/>
+         </geometry>
+       </collision>
+     </link>
+     <joint name="ground_plane_joint" type="fixed">
+       <origin xyz="0 0 -0.01" rpy="0 0 0"/>
+       <parent link="world"/>
+       <child link="ground_plane"/>
+     </joint>
+   </xacro:if>
    <!-- arm -->
    <xacro:ur_robot
@@ -31,10 +86,55 @@
      physical_parameters_file="$(arg physical_params)"
      visual_parameters_file="$(arg visual_params)"
+     transmission_hw_interface="$(arg transmission_hw_interface)"
      safety_limits="$(arg safety_limits)"
      safety_pos_margin="$(arg safety_pos_margin)"
      safety_k_position="$(arg safety_k_position)"
-     force_abs_paths="$(arg force_abs_paths)"
+     use_fake_hardware="$(arg use_fake_hardware)"
+     fake_sensor_commands="$(arg fake_sensor_commands)"
+     sim_gazebo="$(arg sim_gazebo)"
+     sim_ignition="$(arg sim_ignition)"
+     headless_mode="$(arg headless_mode)"
+     initial_positions="${xacro.load_yaml(initial_positions_file)}"
+     use_tool_communication="$(arg use_tool_communication)"
+     tool_voltage="$(arg tool_voltage)"
+     tool_parity="$(arg tool_parity)"
+     tool_baud_rate="$(arg tool_baud_rate)"
+     tool_stop_bits="$(arg tool_stop_bits)"
+     tool_rx_idle_chars="$(arg tool_rx_idle_chars)"
+     tool_tx_idle_chars="$(arg tool_tx_idle_chars)"
+     tool_device_name="$(arg tool_device_name)"
+     tool_tcp_port="$(arg tool_tcp_port)"
+     robot_ip="$(arg robot_ip)"
+     script_filename="$(arg script_filename)"
+     output_recipe_filename="$(arg output_recipe_filename)"
+     input_recipe_filename="$(arg input_recipe_filename)"
+     reverse_ip="$(arg reverse_ip)"
+     script_command_port="$(arg script_command_port)"
+     reverse_port="$(arg reverse_port)"
+     script_sender_port="$(arg script_sender_port)"
+     trajectory_port="$(arg trajectory_port)"
      >
      <origin xyz="0 0 0" rpy="0 0 0" />          <!-- position robot in the world -->
    </xacro:ur_robot>
+   <xacro:if value="$(arg sim_gazebo)">
+    <!-- Gazebo plugins -->
+    <gazebo reference="world">
+    </gazebo>
+    <gazebo>
+      <plugin filename="libgazebo_ros2_control.so" name="gazebo_ros2_control">
+        <parameters>$(arg simulation_controllers)</parameters>
+      </plugin>
+    </gazebo>
+  </xacro:if>
+  <xacro:if value="$(arg sim_ignition)">
+    <!-- Gazebo plugins -->
+    <gazebo reference="world">
+    </gazebo>
+    <gazebo>
+      <plugin filename="libign_ros2_control-system.so" name="ign_ros2_control::IgnitionROS2ControlPlugin">
+        <parameters>$(arg simulation_controllers)</parameters>
+        <controller_manager_node_name>$(arg tf_prefix)controller_manager</controller_manager_node_name>
+      </plugin>
+    </gazebo>
+  </xacro:if>
 </robot>

File: urdf/ur_macro.xacro (robot description, xacro)
@@ -42,4 +42,5 @@
      - Muhammad Asif Rana
   -->
+  <xacro:include filename="$(find ur_description)/urdf/inc/ur_transmissions.xacro" />
   <xacro:include filename="$(find ur_description)/urdf/inc/ur_common.xacro" />
   <xacro:macro name="ur_robot" params="
@@ -52,9 +53,36 @@
     physical_parameters_file
     visual_parameters_file
+    generate_ros2_control_tag:=true
+    transmission_hw_interface:=hardware_interface/PositionJointInterface
     safety_limits:=false
     safety_pos_margin:=0.15
     safety_k_position:=20
-    force_abs_paths:=false
-    ">
+    use_fake_hardware:=false
+    fake_sensor_commands:=false
+    sim_gazebo:=false
+    sim_ignition:=false
+    headless_mode:=false
+    initial_positions:=${dict(shoulder_pan_joint=0.0,shoulder_lift_joint=-1.57,elbow_joint=0.0,wrist_1_joint=-1.57,wrist_2_joint=0.0,wrist_3_joint=0.0)}
+    use_tool_communication:=false
+    tool_voltage:=0
+    tool_parity:=0
+    tool_baud_rate:=115200
+    tool_stop_bits:=1
+    tool_rx_idle_chars:=1.5
+    tool_tx_idle_chars:=3.5
+    tool_device_name:=/tmp/ttyUR
+    tool_tcp_port:=54321
+    robot_ip:=0.0.0.0
+    script_filename:=to_be_filled_by_ur_robot_driver
+    output_recipe_filename:=to_be_filled_by_ur_robot_driver
+    input_recipe_filename:=to_be_filled_by_ur_robot_driver
+    reverse_port:=50001
+    script_sender_port:=50002
+    reverse_ip:=0.0.0.0
+    script_command_port:=50004
+    trajectory_port:=50003
+    non_blocking_read:=true
+    keep_alive_count:=2"
+    >
     <!-- Load configuration data from the provided .yaml files -->
     <xacro:read_model_data
@@ -63,12 +91,45 @@
       physical_parameters_file="${physical_parameters_file}"
       visual_parameters_file="${visual_parameters_file}"
-      force_abs_paths="${force_abs_paths}"/>
+      force_abs_paths="${sim_gazebo or sim_ignition}"/>
+    <xacro:if value="${generate_ros2_control_tag}">
+      <!-- ros2 control include -->
+      <xacro:include filename="$(find ur_description)/urdf/ur.ros2_control.xacro" />
+      <!-- ros2 control instance -->
+      <xacro:ur_ros2_control
+        name="${name}"
+        use_fake_hardware="${use_fake_hardware}"
+        initial_positions="${initial_positions}"
+        fake_sensor_commands="${fake_sensor_commands}"
+        headless_mode="${headless_mode}"
+        sim_gazebo="${sim_gazebo}"
+        sim_ignition="${sim_ignition}"
+        script_filename="${script_filename}"
+        output_recipe_filename="${output_recipe_filename}"
+        input_recipe_filename="${input_recipe_filename}"
+        tf_prefix="${tf_prefix}"
+        hash_kinematics="${kinematics_hash}"
+        robot_ip="${robot_ip}"
+        use_tool_communication="${use_tool_communication}"
+        tool_voltage="${tool_voltage}"
+        tool_parity="${tool_parity}"
+        tool_baud_rate="${tool_baud_rate}"
+        tool_stop_bits="${tool_stop_bits}"
+        tool_rx_idle_chars="${tool_rx_idle_chars}"
+        tool_tx_idle_chars="${tool_tx_idle_chars}"
+        tool_device_name="${tool_device_name}"
+        tool_tcp_port="${tool_tcp_port}"
+        reverse_port="${reverse_port}"
+        script_sender_port="${script_sender_port}"
+        reverse_ip="${reverse_ip}"
+        script_command_port="${script_command_port}"
+        trajectory_port="${trajectory_port}"
+        non_blocking_read="${non_blocking_read}"
+        keep_alive_count="${keep_alive_count}"
+        />
+    </xacro:if>
+    <!-- Add URDF transmission elements (for ros_control) -->
+    <!--<xacro:ur_arm_transmission prefix="${prefix}" hw_interface="${transmission_hw_interface}" />-->
+    <!-- Placeholder for ros2_control transmission which don't yet exist -->
     <!-- links -  main serial chain -->
-    <!-- base_link serves as the root of the robot's kinematic tree. It follows REP-103
-        conventions (i.e., X+ forward, Y+ left, Z+ up).
-        Since some kinematic solvers forbid having inertia values attached to a root link, we've
-        added the base_link_inertia link that carries the visual, collision and inertia
-        information.
-    -->
     <link name="${tf_prefix}base_link"/>
     <link name="${tf_prefix}base_link_inertia">
