Commit message: Imported upstream version '2.4.4' of 'upstream'

File: urdf/ur_macro.xacro (robot description, xacro)
@@ -96,8 +96,16 @@
         </geometry>
       </collision>
-      <xacro:cylinder_inertial radius="${shoulder_inertia_radius}" length="${shoulder_inertia_length}" mass="${shoulder_mass}">
-        <origin xyz="0 0 0" rpy="0 0 0" />
-      </xacro:cylinder_inertial>
-    </link>
+      <inertial>
+        <mass value="${shoulder_mass}"/>
+        <origin rpy="${shoulder_inertia_rotation}" xyz="${shoulder_cog}"/>
+        <inertia
+            ixx="${shoulder_inertia_ixx}"
+            ixy="${shoulder_inertia_ixy}"
+            ixz="${shoulder_inertia_ixz}"
+            iyy="${shoulder_inertia_iyy}"
+            iyz="${shoulder_inertia_iyz}"
+            izz="${shoulder_inertia_izz}"
+        />
+      </inertial>    </link>
     <link name="${tf_prefix}upper_arm_link">
       <visual>
@@ -113,7 +121,16 @@
         </geometry>
       </collision>
-      <xacro:cylinder_inertial radius="${upperarm_inertia_radius}" length="${upperarm_inertia_length}" mass="${upper_arm_mass}">
-        <origin xyz="${-0.5 * upperarm_inertia_length} 0.0 ${upper_arm_inertia_offset}" rpy="0 ${pi/2} 0" />
-      </xacro:cylinder_inertial>
+      <inertial>
+        <mass value="${upper_arm_mass}"/>
+        <origin rpy="${upper_arm_inertia_rotation}" xyz="${upper_arm_cog}"/>
+        <inertia
+            ixx="${upper_arm_inertia_ixx}"
+            ixy="${upper_arm_inertia_ixy}"
+            ixz="${upper_arm_inertia_ixz}"
+            iyy="${upper_arm_inertia_iyy}"
+            iyz="${upper_arm_inertia_iyz}"
+            izz="${upper_arm_inertia_izz}"
+        />
+      </inertial>
     </link>
     <link name="${tf_prefix}forearm_link">
@@ -130,7 +147,16 @@
         </geometry>
       </collision>
-      <xacro:cylinder_inertial radius="${forearm_inertia_radius}" length="${forearm_inertia_length}"  mass="${forearm_mass}">
-        <origin xyz="${-0.5 * forearm_inertia_length} 0.0 ${elbow_offset}" rpy="0 ${pi/2} 0" />
-      </xacro:cylinder_inertial>
+      <inertial>
+        <mass value="${forearm_mass}"/>
+        <origin rpy="${forearm_inertia_rotation}" xyz="${forearm_cog}"/>
+        <inertia
+            ixx="${forearm_inertia_ixx}"
+            ixy="${forearm_inertia_ixy}"
+            ixz="${forearm_inertia_ixz}"
+            iyy="${forearm_inertia_iyy}"
+            iyz="${forearm_inertia_iyz}"
+            izz="${forearm_inertia_izz}"
+        />
+      </inertial>
     </link>
     <link name="${tf_prefix}wrist_1_link">
@@ -148,7 +174,16 @@
         </geometry>
       </collision>
-      <xacro:cylinder_inertial radius="${wrist_1_inertia_radius}" length="${wrist_1_inertia_length}"  mass="${wrist_1_mass}">
-        <origin xyz="0 0 0" rpy="0 0 0" />
-      </xacro:cylinder_inertial>
+      <inertial>
+        <mass value="${wrist_1_mass}"/>
+        <origin rpy="${wrist_1_inertia_rotation}" xyz="${wrist_1_cog}"/>
+        <inertia
+            ixx="${wrist_1_inertia_ixx}"
+            ixy="${wrist_1_inertia_ixy}"
+            ixz="${wrist_1_inertia_ixz}"
+            iyy="${wrist_1_inertia_iyy}"
+            iyz="${wrist_1_inertia_iyz}"
+            izz="${wrist_1_inertia_izz}"
+        />
+      </inertial>
     </link>
     <link name="${tf_prefix}wrist_2_link">
@@ -166,7 +201,16 @@
         </geometry>
       </collision>
-      <xacro:cylinder_inertial radius="${wrist_2_inertia_radius}" length="${wrist_2_inertia_length}"  mass="${wrist_2_mass}">
-        <origin xyz="0 0 0" rpy="0 0 0" />
-      </xacro:cylinder_inertial>
+      <inertial>
+        <mass value="${wrist_2_mass}"/>
+        <origin rpy="${wrist_2_inertia_rotation}" xyz="${wrist_2_cog}"/>
+        <inertia
+            ixx="${wrist_2_inertia_ixx}"
+            ixy="${wrist_2_inertia_ixy}"
+            ixz="${wrist_2_inertia_ixz}"
+            iyy="${wrist_2_inertia_iyy}"
+            iyz="${wrist_2_inertia_iyz}"
+            izz="${wrist_2_inertia_izz}"
+        />
+      </inertial>
     </link>
     <link name="${tf_prefix}wrist_3_link">
@@ -184,7 +228,16 @@
         </geometry>
       </collision>
-      <xacro:cylinder_inertial radius="${wrist_3_inertia_radius}" length="${wrist_3_inertia_length}"  mass="${wrist_3_mass}">
-        <origin xyz="0.0 0.0 ${-0.5 * wrist_3_inertia_length}" rpy="0 0 0" />
-      </xacro:cylinder_inertial>
+      <inertial>
+        <mass value="${wrist_3_mass}"/>
+        <origin rpy="${wrist_3_inertia_rotation}" xyz="${wrist_3_cog}"/>
+        <inertia
+            ixx="${wrist_3_inertia_ixx}"
+            ixy="${wrist_3_inertia_ixy}"
+            ixz="${wrist_3_inertia_ixz}"
+            iyy="${wrist_3_inertia_iyy}"
+            iyz="${wrist_3_inertia_iyz}"
+            izz="${wrist_3_inertia_izz}"
+        />
+      </inertial>
     </link>
     <!-- base_joint fixes base_link to the environment -->
@@ -265,14 +318,22 @@
       <dynamics damping="0" friction="0"/>
     </joint>
-    <joint name="${tf_prefix}wrist_3_joint" type="revolute">
+    <joint name="${tf_prefix}wrist_3_joint" type="${wrist_3_joint_type}">
       <parent link="${tf_prefix}wrist_2_link" />
       <child link="${tf_prefix}wrist_3_link" />
       <origin xyz="${wrist_3_x} ${wrist_3_y} ${wrist_3_z}" rpy="${wrist_3_roll} ${wrist_3_pitch} ${wrist_3_yaw}" />
       <axis xyz="0 0 1" />
-      <limit lower="${wrist_3_lower_limit}" upper="${wrist_3_upper_limit}"
-             effort="${wrist_3_effort_limit}" velocity="${wrist_3_velocity_limit}"/>
-      <xacro:if value="${safety_limits}">
-         <safety_controller soft_lower_limit="${wrist_3_lower_limit + safety_pos_margin}" soft_upper_limit="${wrist_3_upper_limit - safety_pos_margin}" k_position="${safety_k_position}" k_velocity="0.0"/>
-      </xacro:if>
+      <xacro:if value="${wrist_3_joint_type != 'continuous'}">
+        <limit lower="${wrist_3_lower_limit}" upper="${wrist_3_upper_limit}"
+          effort="${wrist_3_effort_limit}" velocity="${wrist_3_velocity_limit}"/>
+        <xacro:if value="${safety_limits}">
+          <safety_controller soft_lower_limit="${wrist_3_lower_limit + safety_pos_margin}" soft_upper_limit="${wrist_3_upper_limit - safety_pos_margin}" k_position="${safety_k_position}" k_velocity="0.0"/>
+        </xacro:if>
+      </xacro:if>
+      <xacro:unless value="${wrist_3_joint_type != 'continuous'}">
+        <limit effort="${wrist_3_effort_limit}" velocity="${wrist_3_velocity_limit}"/>
+        <xacro:if value="${safety_limits}">
+          <safety_controller k_position="${safety_k_position}" k_velocity="0.0"/>
+        </xacro:if>
+      </xacro:unless>
       <dynamics damping="0" friction="0"/>
     </joint>

Commit message: Imported upstream version '3.3.0' of 'upstream'

File: urdf/ur_macro.xacro (robot description, xacro)
@@ -73,9 +73,6 @@
     <link name="${tf_prefix}base_link"/>
     <link name="${tf_prefix}base_link_inertia">
-      <xacro:get_visual_params name="base" type="mesh_offset"/>
-      <visual>
-        <origin
-         xyz="${visual_params['x']} ${visual_params['y']} ${visual_params['z']}"
-         rpy="${visual_params['roll']} ${visual_params['pitch']} ${visual_params['yaw']}"/>
+      <visual>
+        <origin xyz="0 0 0" rpy="0 0 ${pi}"/>
         <geometry>
           <xacro:get_mesh name="base" type="visual"/>
@@ -83,7 +80,5 @@
       </visual>
       <collision>
-        <origin
-         xyz="${visual_params['x']} ${visual_params['y']} ${visual_params['z']}"
-         rpy="${visual_params['roll']} ${visual_params['pitch']} ${visual_params['yaw']}"/>
+        <origin xyz="0 0 0" rpy="0 0 ${pi}"/>
         <geometry>
           <xacro:get_mesh name="base" type="collision"/>
@@ -95,9 +90,6 @@
     </link>
     <link name="${tf_prefix}shoulder_link">
-      <xacro:get_visual_params name="shoulder" type="mesh_offset"/>
-      <visual>
-        <origin
-         xyz="${visual_params['x']} ${visual_params['y']} ${visual_params['z']}"
-         rpy="${visual_params['roll']} ${visual_params['pitch']} ${visual_params['yaw']}"/>
+      <visual>
+        <origin xyz="0 0 0" rpy="0 0 ${pi}"/>
         <geometry>
           <xacro:get_mesh name="shoulder" type="visual"/>
@@ -105,7 +97,5 @@
       </visual>
       <collision>
-        <origin
-         xyz="${visual_params['x']} ${visual_params['y']} ${visual_params['z']}"
-         rpy="${visual_params['roll']} ${visual_params['pitch']} ${visual_params['yaw']}"/>
+        <origin xyz="0 0 0" rpy="0 0 ${pi}"/>
         <geometry>
           <xacro:get_mesh name="shoulder" type="collision"/>
@@ -125,9 +115,6 @@
       </inertial>    </link>
     <link name="${tf_prefix}upper_arm_link">
-      <xacro:get_visual_params name="upper_arm" type="mesh_offset"/>
-      <visual>
-        <origin
-         xyz="${visual_params['x']} ${visual_params['y']} ${visual_params['z']}"
-         rpy="${visual_params['roll']} ${visual_params['pitch']} ${visual_params['yaw']}"/>
+      <visual>
+        <origin xyz="0 0 ${shoulder_offset}" rpy="${pi/2} 0 ${-pi/2}"/>
         <geometry>
           <xacro:get_mesh name="upper_arm" type="visual"/>
@@ -135,7 +122,5 @@
       </visual>
       <collision>
-        <origin
-         xyz="${visual_params['x']} ${visual_params['y']} ${visual_params['z']}"
-         rpy="${visual_params['roll']} ${visual_params['pitch']} ${visual_params['yaw']}"/>
+        <origin xyz="0 0 ${shoulder_offset}" rpy="${pi/2} 0 ${-pi/2}"/>
         <geometry>
           <xacro:get_mesh name="upper_arm" type="collision"/>
@@ -156,9 +141,6 @@
     </link>
     <link name="${tf_prefix}forearm_link">
-      <xacro:get_visual_params name="forearm" type="mesh_offset"/>
-      <visual>
-        <origin
-         xyz="${visual_params['x']} ${visual_params['y']} ${visual_params['z']}"
-         rpy="${visual_params['roll']} ${visual_params['pitch']} ${visual_params['yaw']}"/>
+      <visual>
+        <origin xyz="0 0 ${elbow_offset}" rpy="${pi/2} 0 ${-pi/2}"/>
         <geometry>
           <xacro:get_mesh name="forearm" type="visual"/>
@@ -166,7 +148,5 @@
       </visual>
       <collision>
-        <origin
-         xyz="${visual_params['x']} ${visual_params['y']} ${visual_params['z']}"
-         rpy="${visual_params['roll']} ${visual_params['pitch']} ${visual_params['yaw']}"/>
+        <origin xyz="0 0 ${elbow_offset}" rpy="${pi/2} 0 ${-pi/2}"/>
         <geometry>
           <xacro:get_mesh name="forearm" type="collision"/>
@@ -187,9 +167,7 @@
     </link>
     <link name="${tf_prefix}wrist_1_link">
-      <xacro:get_visual_params name="wrist_1" type="mesh_offset"/>
-      <visual>
-        <origin
-         xyz="${visual_params['x']} ${visual_params['y']} ${visual_params['z']}"
-         rpy="${visual_params['roll']} ${visual_params['pitch']} ${visual_params['yaw']}"/>
+	  <xacro:get_visual_params name="wrist_1" type="visual_offset"/>
+      <visual>
+      	<origin xyz="0 0 ${visual_params}" rpy="${pi/2} 0 0"/>
         <geometry>
           <xacro:get_mesh name="wrist_1" type="visual"/>
@@ -197,7 +175,5 @@
       </visual>
       <collision>
-        <origin
-         xyz="${visual_params['x']} ${visual_params['y']} ${visual_params['z']}"
-         rpy="${visual_params['roll']} ${visual_params['pitch']} ${visual_params['yaw']}"/>
+        <origin xyz="0 0 ${visual_params}" rpy="${pi/2} 0 0"/>
         <geometry>
           <xacro:get_mesh name="wrist_1" type="collision"/>
@@ -218,9 +194,7 @@
     </link>
     <link name="${tf_prefix}wrist_2_link">
-      <xacro:get_visual_params name="wrist_2" type="mesh_offset"/>
-      <visual>
-        <origin
-         xyz="${visual_params['x']} ${visual_params['y']} ${visual_params['z']}"
-         rpy="${visual_params['roll']} ${visual_params['pitch']} ${visual_params['yaw']}"/>
+          <xacro:get_visual_params name="wrist_2" type="visual_offset"/>
+      <visual>
+        <origin xyz="0 0 ${visual_params}" rpy="0 0 0"/>
         <geometry>
           <xacro:get_mesh name="wrist_2" type="visual"/>
@@ -228,7 +202,5 @@
       </visual>
       <collision>
-        <origin
-         xyz="${visual_params['x']} ${visual_params['y']} ${visual_params['z']}"
-         rpy="${visual_params['roll']} ${visual_params['pitch']} ${visual_params['yaw']}"/>
+        <origin xyz="0 0 ${visual_params}" rpy="0 0 0"/>
         <geometry>
           <xacro:get_mesh name="wrist_2" type="collision"/>
@@ -249,9 +221,13 @@
     </link>
     <link name="${tf_prefix}wrist_3_link">
-      <xacro:get_visual_params name="wrist_3" type="mesh_offset"/>
-      <visual>
-        <origin
-         xyz="${visual_params['x']} ${visual_params['y']} ${visual_params['z']}"
-         rpy="${visual_params['roll']} ${visual_params['pitch']} ${visual_params['yaw']}"/>
+      <!-- TODO: remove this once all wrist_3 meshes have the visual_offset_xyz tag -->
+      <xacro:get_visual_params name="wrist_3" type="visual_offset_xyz"/>
+      <xacro:property name="mesh_offset" value="${visual_params}" scope="parent"/>
+      <xacro:if value="${visual_params == ''}">
+        <xacro:get_visual_params name="wrist_3" type="visual_offset"/>
+        <xacro:property name="mesh_offset" value="0 0 ${visual_params}" scope="parent"/>
+      </xacro:if>
+      <visual>
+        <origin xyz="${mesh_offset}" rpy="${pi/2} 0 0"/>
         <geometry>
           <xacro:get_mesh name="wrist_3" type="visual"/>
@@ -259,7 +235,5 @@
       </visual>
       <collision>
-        <origin
-         xyz="${visual_params['x']} ${visual_params['y']} ${visual_params['z']}"
-         rpy="${visual_params['roll']} ${visual_params['pitch']} ${visual_params['yaw']}"/>
+        <origin xyz="${mesh_offset}" rpy="${pi/2} 0 0"/>
         <geometry>
           <xacro:get_mesh name="wrist_3" type="collision"/>

Commit message: Imported upstream version '4.1.1' of 'upstream'

File: urdf/ur_macro.xacro (robot description, xacro)
@@ -73,6 +73,9 @@
     <link name="${tf_prefix}base_link"/>
     <link name="${tf_prefix}base_link_inertia">
-      <visual>
-        <origin xyz="0 0 0" rpy="0 0 ${pi}"/>
+      <xacro:get_visual_params name="base" type="mesh_offset"/>
+      <visual>
+        <origin
+         xyz="${visual_params['x']} ${visual_params['y']} ${visual_params['z']}"
+         rpy="${visual_params['roll']} ${visual_params['pitch']} ${visual_params['yaw']}"/>
         <geometry>
           <xacro:get_mesh name="base" type="visual"/>
@@ -80,5 +83,7 @@
       </visual>
       <collision>
-        <origin xyz="0 0 0" rpy="0 0 ${pi}"/>
+        <origin
+         xyz="${visual_params['x']} ${visual_params['y']} ${visual_params['z']}"
+         rpy="${visual_params['roll']} ${visual_params['pitch']} ${visual_params['yaw']}"/>
         <geometry>
           <xacro:get_mesh name="base" type="collision"/>
@@ -90,6 +95,9 @@
     </link>
     <link name="${tf_prefix}shoulder_link">
-      <visual>
-        <origin xyz="0 0 0" rpy="0 0 ${pi}"/>
+      <xacro:get_visual_params name="shoulder" type="mesh_offset"/>
+      <visual>
+        <origin
+         xyz="${visual_params['x']} ${visual_params['y']} ${visual_params['z']}"
+         rpy="${visual_params['roll']} ${visual_params['pitch']} ${visual_params['yaw']}"/>
         <geometry>
           <xacro:get_mesh name="shoulder" type="visual"/>
@@ -97,5 +105,7 @@
       </visual>
       <collision>
-        <origin xyz="0 0 0" rpy="0 0 ${pi}"/>
+        <origin
+         xyz="${visual_params['x']} ${visual_params['y']} ${visual_params['z']}"
+         rpy="${visual_params['roll']} ${visual_params['pitch']} ${visual_params['yaw']}"/>
         <geometry>
           <xacro:get_mesh name="shoulder" type="collision"/>
@@ -115,6 +125,9 @@
       </inertial>    </link>
     <link name="${tf_prefix}upper_arm_link">
-      <visual>
-        <origin xyz="0 0 ${shoulder_offset}" rpy="${pi/2} 0 ${-pi/2}"/>
+      <xacro:get_visual_params name="upper_arm" type="mesh_offset"/>
+      <visual>
+        <origin
+         xyz="${visual_params['x']} ${visual_params['y']} ${visual_params['z']}"
+         rpy="${visual_params['roll']} ${visual_params['pitch']} ${visual_params['yaw']}"/>
         <geometry>
           <xacro:get_mesh name="upper_arm" type="visual"/>
@@ -122,5 +135,7 @@
       </visual>
       <collision>
-        <origin xyz="0 0 ${shoulder_offset}" rpy="${pi/2} 0 ${-pi/2}"/>
+        <origin
+         xyz="${visual_params['x']} ${visual_params['y']} ${visual_params['z']}"
+         rpy="${visual_params['roll']} ${visual_params['pitch']} ${visual_params['yaw']}"/>
         <geometry>
           <xacro:get_mesh name="upper_arm" type="collision"/>
@@ -141,6 +156,9 @@
     </link>
     <link name="${tf_prefix}forearm_link">
-      <visual>
-        <origin xyz="0 0 ${elbow_offset}" rpy="${pi/2} 0 ${-pi/2}"/>
+      <xacro:get_visual_params name="forearm" type="mesh_offset"/>
+      <visual>
+        <origin
+         xyz="${visual_params['x']} ${visual_params['y']} ${visual_params['z']}"
+         rpy="${visual_params['roll']} ${visual_params['pitch']} ${visual_params['yaw']}"/>
         <geometry>
           <xacro:get_mesh name="forearm" type="visual"/>
@@ -148,5 +166,7 @@
       </visual>
       <collision>
-        <origin xyz="0 0 ${elbow_offset}" rpy="${pi/2} 0 ${-pi/2}"/>
+        <origin
+         xyz="${visual_params['x']} ${visual_params['y']} ${visual_params['z']}"
+         rpy="${visual_params['roll']} ${visual_params['pitch']} ${visual_params['yaw']}"/>
         <geometry>
           <xacro:get_mesh name="forearm" type="collision"/>
@@ -167,7 +187,9 @@
     </link>
     <link name="${tf_prefix}wrist_1_link">
-	  <xacro:get_visual_params name="wrist_1" type="visual_offset"/>
-      <visual>
-      	<origin xyz="0 0 ${visual_params}" rpy="${pi/2} 0 0"/>
+      <xacro:get_visual_params name="wrist_1" type="mesh_offset"/>
+      <visual>
+        <origin
+         xyz="${visual_params['x']} ${visual_params['y']} ${visual_params['z']}"
+         rpy="${visual_params['roll']} ${visual_params['pitch']} ${visual_params['yaw']}"/>
         <geometry>
           <xacro:get_mesh name="wrist_1" type="visual"/>
@@ -175,5 +197,7 @@
       </visual>
       <collision>
-        <origin xyz="0 0 ${visual_params}" rpy="${pi/2} 0 0"/>
+        <origin
+         xyz="${visual_params['x']} ${visual_params['y']} ${visual_params['z']}"
+         rpy="${visual_params['roll']} ${visual_params['pitch']} ${visual_params['yaw']}"/>
         <geometry>
           <xacro:get_mesh name="wrist_1" type="collision"/>
@@ -194,7 +218,9 @@
     </link>
     <link name="${tf_prefix}wrist_2_link">
-          <xacro:get_visual_params name="wrist_2" type="visual_offset"/>
-      <visual>
-        <origin xyz="0 0 ${visual_params}" rpy="0 0 0"/>
+      <xacro:get_visual_params name="wrist_2" type="mesh_offset"/>
+      <visual>
+        <origin
+         xyz="${visual_params['x']} ${visual_params['y']} ${visual_params['z']}"
+         rpy="${visual_params['roll']} ${visual_params['pitch']} ${visual_params['yaw']}"/>
         <geometry>
           <xacro:get_mesh name="wrist_2" type="visual"/>
@@ -202,5 +228,7 @@
       </visual>
       <collision>
-        <origin xyz="0 0 ${visual_params}" rpy="0 0 0"/>
+        <origin
+         xyz="${visual_params['x']} ${visual_params['y']} ${visual_params['z']}"
+         rpy="${visual_params['roll']} ${visual_params['pitch']} ${visual_params['yaw']}"/>
         <geometry>
           <xacro:get_mesh name="wrist_2" type="collision"/>
@@ -221,13 +249,9 @@
     </link>
     <link name="${tf_prefix}wrist_3_link">
-      <!-- TODO: remove this once all wrist_3 meshes have the visual_offset_xyz tag -->
-      <xacro:get_visual_params name="wrist_3" type="visual_offset_xyz"/>
-      <xacro:property name="mesh_offset" value="${visual_params}" scope="parent"/>
-      <xacro:if value="${visual_params == ''}">
-        <xacro:get_visual_params name="wrist_3" type="visual_offset"/>
-        <xacro:property name="mesh_offset" value="0 0 ${visual_params}" scope="parent"/>
-      </xacro:if>
-      <visual>
-        <origin xyz="${mesh_offset}" rpy="${pi/2} 0 0"/>
+      <xacro:get_visual_params name="wrist_3" type="mesh_offset"/>
+      <visual>
+        <origin
+         xyz="${visual_params['x']} ${visual_params['y']} ${visual_params['z']}"
+         rpy="${visual_params['roll']} ${visual_params['pitch']} ${visual_params['yaw']}"/>
         <geometry>
           <xacro:get_mesh name="wrist_3" type="visual"/>
@@ -235,5 +259,7 @@
       </visual>
       <collision>
-        <origin xyz="${mesh_offset}" rpy="${pi/2} 0 0"/>
+        <origin
+         xyz="${visual_params['x']} ${visual_params['y']} ${visual_params['z']}"
+         rpy="${visual_params['roll']} ${visual_params['pitch']} ${visual_params['yaw']}"/>
         <geometry>
           <xacro:get_mesh name="wrist_3" type="collision"/>
