Commit message: Imported upstream version '2.10.1' of 'upstream'

File: urdf/ur_macro.xacro (robot description, xacro)
@@ -42,4 +42,5 @@
      - Muhammad Asif Rana
   -->
+  <xacro:include filename="$(find ur_description)/urdf/inc/ur_transmissions.xacro" />
   <xacro:include filename="$(find ur_description)/urdf/inc/ur_common.xacro" />
   <xacro:macro name="ur_robot" params="
@@ -52,9 +53,36 @@
     physical_parameters_file
     visual_parameters_file
+    generate_ros2_control_tag:=true
+    transmission_hw_interface:=hardware_interface/PositionJointInterface
     safety_limits:=false
     safety_pos_margin:=0.15
     safety_k_position:=20
-    force_abs_paths:=false
-    ">
+    use_fake_hardware:=false
+    fake_sensor_commands:=false
+    sim_gazebo:=false
+    sim_ignition:=false
+    headless_mode:=false
+    initial_positions:=${dict(shoulder_pan_joint=0.0,shoulder_lift_joint=-1.57,elbow_joint=0.0,wrist_1_joint=-1.57,wrist_2_joint=0.0,wrist_3_joint=0.0)}
+    use_tool_communication:=false
+    tool_voltage:=0
+    tool_parity:=0
+    tool_baud_rate:=115200
+    tool_stop_bits:=1
+    tool_rx_idle_chars:=1.5
+    tool_tx_idle_chars:=3.5
+    tool_device_name:=/tmp/ttyUR
+    tool_tcp_port:=54321
+    robot_ip:=0.0.0.0
+    script_filename:=to_be_filled_by_ur_robot_driver
+    output_recipe_filename:=to_be_filled_by_ur_robot_driver
+    input_recipe_filename:=to_be_filled_by_ur_robot_driver
+    reverse_port:=50001
+    script_sender_port:=50002
+    reverse_ip:=0.0.0.0
+    script_command_port:=50004
+    trajectory_port:=50003
+    non_blocking_read:=true
+    keep_alive_count:=2"
+    >
     <!-- Load configuration data from the provided .yaml files -->
     <xacro:read_model_data
@@ -63,19 +91,49 @@
       physical_parameters_file="${physical_parameters_file}"
       visual_parameters_file="${visual_parameters_file}"
-      force_abs_paths="${force_abs_paths}"/>
+      force_abs_paths="${sim_gazebo or sim_ignition}"/>
+    <xacro:if value="${generate_ros2_control_tag}">
+      <!-- ros2 control include -->
+      <xacro:include filename="$(find ur_description)/urdf/ur.ros2_control.xacro" />
+      <!-- ros2 control instance -->
+      <xacro:ur_ros2_control
+        name="${name}"
+        use_fake_hardware="${use_fake_hardware}"
+        initial_positions="${initial_positions}"
+        fake_sensor_commands="${fake_sensor_commands}"
+        headless_mode="${headless_mode}"
+        sim_gazebo="${sim_gazebo}"
+        sim_ignition="${sim_ignition}"
+        script_filename="${script_filename}"
+        output_recipe_filename="${output_recipe_filename}"
+        input_recipe_filename="${input_recipe_filename}"
+        tf_prefix="${tf_prefix}"
+        hash_kinematics="${kinematics_hash}"
+        robot_ip="${robot_ip}"
+        use_tool_communication="${use_tool_communication}"
+        tool_voltage="${tool_voltage}"
+        tool_parity="${tool_parity}"
+        tool_baud_rate="${tool_baud_rate}"
+        tool_stop_bits="${tool_stop_bits}"
+        tool_rx_idle_chars="${tool_rx_idle_chars}"
+        tool_tx_idle_chars="${tool_tx_idle_chars}"
+        tool_device_name="${tool_device_name}"
+        tool_tcp_port="${tool_tcp_port}"
+        reverse_port="${reverse_port}"
+        script_sender_port="${script_sender_port}"
+        reverse_ip="${reverse_ip}"
+        script_command_port="${script_command_port}"
+        trajectory_port="${trajectory_port}"
+        non_blocking_read="${non_blocking_read}"
+        keep_alive_count="${keep_alive_count}"
+        />
+    </xacro:if>
+    <!-- Add URDF transmission elements (for ros_control) -->
+    <!--<xacro:ur_arm_transmission prefix="${prefix}" hw_interface="${transmission_hw_interface}" />-->
+    <!-- Placeholder for ros2_control transmission which don't yet exist -->
     <!-- links -  main serial chain -->
-    <!-- base_link serves as the root of the robot's kinematic tree. It follows REP-103
-        conventions (i.e., X+ forward, Y+ left, Z+ up).
-        Since some kinematic solvers forbid having inertia values attached to a root link, we've
-        added the base_link_inertia link that carries the visual, collision and inertia
-        information.
-    -->
     <link name="${tf_prefix}base_link"/>
     <link name="${tf_prefix}base_link_inertia">
-      <xacro:get_visual_params name="base" type="mesh_offset"/>
-      <visual>
-        <origin
-         xyz="${visual_params['x']} ${visual_params['y']} ${visual_params['z']}"
-         rpy="${visual_params['roll']} ${visual_params['pitch']} ${visual_params['yaw']}"/>
+      <visual>
+        <origin xyz="0 0 0" rpy="0 0 ${pi}"/>
         <geometry>
           <xacro:get_mesh name="base" type="visual"/>
@@ -83,7 +141,5 @@
       </visual>
       <collision>
-        <origin
-         xyz="${visual_params['x']} ${visual_params['y']} ${visual_params['z']}"
-         rpy="${visual_params['roll']} ${visual_params['pitch']} ${visual_params['yaw']}"/>
+        <origin xyz="0 0 0" rpy="0 0 ${pi}"/>
         <geometry>
           <xacro:get_mesh name="base" type="collision"/>
@@ -95,9 +151,6 @@
     </link>
     <link name="${tf_prefix}shoulder_link">
-      <xacro:get_visual_params name="shoulder" type="mesh_offset"/>
-      <visual>
-        <origin
-         xyz="${visual_params['x']} ${visual_params['y']} ${visual_params['z']}"
-         rpy="${visual_params['roll']} ${visual_params['pitch']} ${visual_params['yaw']}"/>
+      <visual>
+        <origin xyz="0 0 0" rpy="0 0 ${pi}"/>
         <geometry>
           <xacro:get_mesh name="shoulder" type="visual"/>
@@ -105,7 +158,5 @@
       </visual>
       <collision>
-        <origin
-         xyz="${visual_params['x']} ${visual_params['y']} ${visual_params['z']}"
-         rpy="${visual_params['roll']} ${visual_params['pitch']} ${visual_params['yaw']}"/>
+        <origin xyz="0 0 0" rpy="0 0 ${pi}"/>
         <geometry>
           <xacro:get_mesh name="shoulder" type="collision"/>
@@ -125,9 +176,6 @@
       </inertial>    </link>
     <link name="${tf_prefix}upper_arm_link">
-      <xacro:get_visual_params name="upper_arm" type="mesh_offset"/>
-      <visual>
-        <origin
-         xyz="${visual_params['x']} ${visual_params['y']} ${visual_params['z']}"
-         rpy="${visual_params['roll']} ${visual_params['pitch']} ${visual_params['yaw']}"/>
+      <visual>
+        <origin xyz="0 0 ${shoulder_offset}" rpy="${pi/2} 0 ${-pi/2}"/>
         <geometry>
           <xacro:get_mesh name="upper_arm" type="visual"/>
@@ -135,7 +183,5 @@
       </visual>
       <collision>
-        <origin
-         xyz="${visual_params['x']} ${visual_params['y']} ${visual_params['z']}"
-         rpy="${visual_params['roll']} ${visual_params['pitch']} ${visual_params['yaw']}"/>
+        <origin xyz="0 0 ${shoulder_offset}" rpy="${pi/2} 0 ${-pi/2}"/>
         <geometry>
           <xacro:get_mesh name="upper_arm" type="collision"/>
@@ -156,9 +202,6 @@
     </link>
     <link name="${tf_prefix}forearm_link">
-      <xacro:get_visual_params name="forearm" type="mesh_offset"/>
-      <visual>
-        <origin
-         xyz="${visual_params['x']} ${visual_params['y']} ${visual_params['z']}"
-         rpy="${visual_params['roll']} ${visual_params['pitch']} ${visual_params['yaw']}"/>
+      <visual>
+        <origin xyz="0 0 ${elbow_offset}" rpy="${pi/2} 0 ${-pi/2}"/>
         <geometry>
           <xacro:get_mesh name="forearm" type="visual"/>
@@ -166,7 +209,5 @@
       </visual>
       <collision>
-        <origin
-         xyz="${visual_params['x']} ${visual_params['y']} ${visual_params['z']}"
-         rpy="${visual_params['roll']} ${visual_params['pitch']} ${visual_params['yaw']}"/>
+        <origin xyz="0 0 ${elbow_offset}" rpy="${pi/2} 0 ${-pi/2}"/>
         <geometry>
           <xacro:get_mesh name="forearm" type="collision"/>
@@ -187,9 +228,7 @@
     </link>
     <link name="${tf_prefix}wrist_1_link">
-      <xacro:get_visual_params name="wrist_1" type="mesh_offset"/>
-      <visual>
-        <origin
-         xyz="${visual_params['x']} ${visual_params['y']} ${visual_params['z']}"
-         rpy="${visual_params['roll']} ${visual_params['pitch']} ${visual_params['yaw']}"/>
+	  <xacro:get_visual_params name="wrist_1" type="visual_offset"/>
+      <visual>
+      	<origin xyz="0 0 ${visual_params}" rpy="${pi/2} 0 0"/>
         <geometry>
           <xacro:get_mesh name="wrist_1" type="visual"/>
@@ -197,7 +236,5 @@
       </visual>
       <collision>
-        <origin
-         xyz="${visual_params['x']} ${visual_params['y']} ${visual_params['z']}"
-         rpy="${visual_params['roll']} ${visual_params['pitch']} ${visual_params['yaw']}"/>
+        <origin xyz="0 0 ${visual_params}" rpy="${pi/2} 0 0"/>
         <geometry>
           <xacro:get_mesh name="wrist_1" type="collision"/>
@@ -218,9 +255,7 @@
     </link>
     <link name="${tf_prefix}wrist_2_link">
-      <xacro:get_visual_params name="wrist_2" type="mesh_offset"/>
-      <visual>
-        <origin
-         xyz="${visual_params['x']} ${visual_params['y']} ${visual_params['z']}"
-         rpy="${visual_params['roll']} ${visual_params['pitch']} ${visual_params['yaw']}"/>
+          <xacro:get_visual_params name="wrist_2" type="visual_offset"/>
+      <visual>
+        <origin xyz="0 0 ${visual_params}" rpy="0 0 0"/>
         <geometry>
           <xacro:get_mesh name="wrist_2" type="visual"/>
@@ -228,7 +263,5 @@
       </visual>
       <collision>
-        <origin
-         xyz="${visual_params['x']} ${visual_params['y']} ${visual_params['z']}"
-         rpy="${visual_params['roll']} ${visual_params['pitch']} ${visual_params['yaw']}"/>
+        <origin xyz="0 0 ${visual_params}" rpy="0 0 0"/>
         <geometry>
           <xacro:get_mesh name="wrist_2" type="collision"/>
@@ -249,9 +282,13 @@
     </link>
     <link name="${tf_prefix}wrist_3_link">
-      <xacro:get_visual_params name="wrist_3" type="mesh_offset"/>
-      <visual>
-        <origin
-         xyz="${visual_params['x']} ${visual_params['y']} ${visual_params['z']}"
-         rpy="${visual_params['roll']} ${visual_params['pitch']} ${visual_params['yaw']}"/>
+      <!-- TODO: remove this once all wrist_3 meshes have the visual_offset_xyz tag -->
+      <xacro:get_visual_params name="wrist_3" type="visual_offset_xyz"/>
+      <xacro:property name="mesh_offset" value="${visual_params}" scope="parent"/>
+      <xacro:if value="${visual_params == ''}">
+        <xacro:get_visual_params name="wrist_3" type="visual_offset"/>
+        <xacro:property name="mesh_offset" value="0 0 ${visual_params}" scope="parent"/>
+      </xacro:if>
+      <visual>
+        <origin xyz="${mesh_offset}" rpy="${pi/2} 0 0"/>
         <geometry>
           <xacro:get_mesh name="wrist_3" type="visual"/>
@@ -259,7 +296,5 @@
       </visual>
       <collision>
-        <origin
-         xyz="${visual_params['x']} ${visual_params['y']} ${visual_params['z']}"
-         rpy="${visual_params['roll']} ${visual_params['pitch']} ${visual_params['yaw']}"/>
+        <origin xyz="${mesh_offset}" rpy="${pi/2} 0 0"/>
         <geometry>
           <xacro:get_mesh name="wrist_3" type="collision"/>
