Commit message: Imported upstream version '2.15.0' of 'upstream'

File: urdf/ur_macro.xacro (robot description, xacro)
@@ -86,5 +86,6 @@
     keep_alive_count:=2
     verify_robot_model:=false
-    use_currents_as_efforts:=true"
+    use_currents_as_efforts:=true
+    smart_panel:=''"
     >
     <!-- Load configuration data from the provided .yaml files -->
@@ -137,9 +138,11 @@
     <!--<xacro:ur_arm_transmission prefix="${prefix}" hw_interface="${transmission_hw_interface}" />-->
     <!-- Placeholder for ros2_control transmission which don't yet exist -->
+    <!-- Empty smart_panel argument means "use visual_parameters.yaml". -->
+    <xacro:property name="smart_panel_enabled" value="${smart_panel if smart_panel != '' else smart_panel_from_visual}"/>
     <!-- links -  main serial chain -->
     <link name="${tf_prefix}base_link"/>
     <link name="${tf_prefix}base_link_inertia">
       <visual>
-        <origin xyz="0 0 0" rpy="0 0 ${pi}"/>
+        <xacro:mesh_origin name="base" legacy_xyz="0 0 0" legacy_rpy="0 0 ${pi}"/>
         <geometry>
           <xacro:get_mesh name="base" type="visual"/>
@@ -147,5 +150,5 @@
       </visual>
       <collision>
-        <origin xyz="0 0 0" rpy="0 0 ${pi}"/>
+        <xacro:mesh_origin name="base" legacy_xyz="0 0 0" legacy_rpy="0 0 ${pi}"/>
         <geometry>
           <xacro:get_mesh name="base" type="collision"/>
@@ -158,5 +161,5 @@
     <link name="${tf_prefix}shoulder_link">
       <visual>
-        <origin xyz="0 0 0" rpy="0 0 ${pi}"/>
+        <xacro:mesh_origin name="shoulder" legacy_xyz="0 0 0" legacy_rpy="0 0 ${pi}"/>
         <geometry>
           <xacro:get_mesh name="shoulder" type="visual"/>
@@ -164,5 +167,5 @@
       </visual>
       <collision>
-        <origin xyz="0 0 0" rpy="0 0 ${pi}"/>
+        <xacro:mesh_origin name="shoulder" legacy_xyz="0 0 0" legacy_rpy="0 0 ${pi}"/>
         <geometry>
           <xacro:get_mesh name="shoulder" type="collision"/>
@@ -183,5 +186,5 @@
     <link name="${tf_prefix}upper_arm_link">
       <visual>
-        <origin xyz="0 0 ${shoulder_offset}" rpy="${pi/2} 0 ${-pi/2}"/>
+        <xacro:mesh_origin name="upper_arm" legacy_xyz="0 0 ${shoulder_offset}" legacy_rpy="${pi/2} 0 ${-pi/2}"/>
         <geometry>
           <xacro:get_mesh name="upper_arm" type="visual"/>
@@ -189,5 +192,5 @@
       </visual>
       <collision>
-        <origin xyz="0 0 ${shoulder_offset}" rpy="${pi/2} 0 ${-pi/2}"/>
+        <xacro:mesh_origin name="upper_arm" legacy_xyz="0 0 ${shoulder_offset}" legacy_rpy="${pi/2} 0 ${-pi/2}"/>
         <geometry>
           <xacro:get_mesh name="upper_arm" type="collision"/>
@@ -209,5 +212,5 @@
     <link name="${tf_prefix}forearm_link">
       <visual>
-        <origin xyz="0 0 ${elbow_offset}" rpy="${pi/2} 0 ${-pi/2}"/>
+        <xacro:mesh_origin name="forearm" legacy_xyz="0 0 ${elbow_offset}" legacy_rpy="${pi/2} 0 ${-pi/2}"/>
         <geometry>
           <xacro:get_mesh name="forearm" type="visual"/>
@@ -215,5 +218,5 @@
       </visual>
       <collision>
-        <origin xyz="0 0 ${elbow_offset}" rpy="${pi/2} 0 ${-pi/2}"/>
+        <xacro:mesh_origin name="forearm" legacy_xyz="0 0 ${elbow_offset}" legacy_rpy="${pi/2} 0 ${-pi/2}"/>
         <geometry>
           <xacro:get_mesh name="forearm" type="collision"/>
@@ -234,7 +237,8 @@
     </link>
     <link name="${tf_prefix}wrist_1_link">
-	  <xacro:get_visual_params name="wrist_1" type="visual_offset"/>
-      <visual>
-      	<origin xyz="0 0 ${visual_params}" rpy="${pi/2} 0 0"/>
+      <xacro:get_visual_params name="wrist_1" type="visual_offset"/>
+      <xacro:property name="wrist_1_legacy_offset" value="${visual_params}"/>
+      <visual>
+        <xacro:mesh_origin name="wrist_1" legacy_xyz="0 0 ${wrist_1_legacy_offset}" legacy_rpy="${pi/2} 0 0"/>
         <geometry>
           <xacro:get_mesh name="wrist_1" type="visual"/>
@@ -242,5 +246,5 @@
       </visual>
       <collision>
-        <origin xyz="0 0 ${visual_params}" rpy="${pi/2} 0 0"/>
+        <xacro:mesh_origin name="wrist_1" legacy_xyz="0 0 ${wrist_1_legacy_offset}" legacy_rpy="${pi/2} 0 0"/>
         <geometry>
           <xacro:get_mesh name="wrist_1" type="collision"/>
@@ -261,7 +265,8 @@
     </link>
     <link name="${tf_prefix}wrist_2_link">
-          <xacro:get_visual_params name="wrist_2" type="visual_offset"/>
-      <visual>
-        <origin xyz="0 0 ${visual_params}" rpy="0 0 0"/>
+      <xacro:get_visual_params name="wrist_2" type="visual_offset"/>
+      <xacro:property name="wrist_2_legacy_offset" value="${visual_params}"/>
+      <visual>
+        <xacro:mesh_origin name="wrist_2" legacy_xyz="0 0 ${wrist_2_legacy_offset}" legacy_rpy="0 0 0"/>
         <geometry>
           <xacro:get_mesh name="wrist_2" type="visual"/>
@@ -269,5 +274,5 @@
       </visual>
       <collision>
-        <origin xyz="0 0 ${visual_params}" rpy="0 0 0"/>
+        <xacro:mesh_origin name="wrist_2" legacy_xyz="0 0 ${wrist_2_legacy_offset}" legacy_rpy="0 0 0"/>
         <geometry>
           <xacro:get_mesh name="wrist_2" type="collision"/>
@@ -296,5 +301,5 @@
       </xacro:if>
       <visual>
-        <origin xyz="${mesh_offset}" rpy="${pi/2} 0 0"/>
+        <xacro:mesh_origin name="wrist_3" legacy_xyz="${mesh_offset}" legacy_rpy="${pi/2} 0 0"/>
         <geometry>
           <xacro:get_mesh name="wrist_3" type="visual"/>
@@ -302,5 +307,5 @@
       </visual>
       <collision>
-        <origin xyz="${mesh_offset}" rpy="${pi/2} 0 0"/>
+        <xacro:mesh_origin name="wrist_3" legacy_xyz="${mesh_offset}" legacy_rpy="${pi/2} 0 0"/>
         <geometry>
           <xacro:get_mesh name="wrist_3" type="collision"/>
@@ -442,4 +447,45 @@
       <origin xyz="0 0 0" rpy="0 ${-pi/2.0} ${-pi/2.0}" />
     </joint>
+    <!-- Optional Smart Panel accessory attached to wrist_3_link.
+         Geometry lives in meshes/common/smart_panel so it can be reused
+         across robot models. -->
+    <xacro:if value="${smart_panel_enabled}">
+      <xacro:if value="${force_abs_paths}">
+        <xacro:property name="smart_panel_visual_mesh" value="file://$(find ur_description)/meshes/common/smart_panel/visual/smart_panel.dae"/>
+        <xacro:property name="smart_panel_collision_mesh" value="file://$(find ur_description)/meshes/common/smart_panel/collision/smart_panel.stl"/>
+      </xacro:if>
+      <xacro:unless value="${force_abs_paths}">
+        <xacro:property name="smart_panel_visual_mesh" value="package://ur_description/meshes/common/smart_panel/visual/smart_panel.dae"/>
+        <xacro:property name="smart_panel_collision_mesh" value="package://ur_description/meshes/common/smart_panel/collision/smart_panel.stl"/>
+      </xacro:unless>
+      <link name="${tf_prefix}smart_panel">
+        <visual>
+          <origin xyz="0 0 0" rpy="0 0 0"/>
+          <geometry>
+            <mesh filename="${smart_panel_visual_mesh}"/>
+          </geometry>
+        </visual>
+        <collision>
+          <origin xyz="0 0 0" rpy="0 0 0"/>
+          <geometry>
+            <mesh filename="${smart_panel_collision_mesh}"/>
+          </geometry>
+        </collision>
+        <inertial>
+          <!-- Inertia estimated for homogeneous weight distribution and the measured mass of the smart panel. -->
+          <origin xyz="0.045 0 -0.030" rpy="0 0 0"/>
+          <mass value="0.0195"/>
+          <inertia ixx="5.682064e-06" ixy="4.66603e-10" ixz="1.863097e-07"
+                   iyy="3.330845e-06" iyz="-2.165772e-09"
+                   izz="3.256972e-06"/>
+        </inertial>
+      </link>
+      <joint name="${tf_prefix}wrist_3_link-smart_panel" type="fixed">
+        <parent link="${tf_prefix}wrist_3_link"/>
+        <child link="${tf_prefix}smart_panel"/>
+        <!-- the mesh is in the correct position relative to wrist_3_link -->
+        <origin xyz="0 0 0" rpy="0 0 0"/>
+      </joint>
+    </xacro:if>
     <!-- ROS-Industrial 'tool0' frame - all-zeros tool frame -->
     <link name="${tf_prefix}tool0"/>
