Commit message: Rebase from 'debian/jazzy/ur_description'

File: urdf/inc/ur_common.xacro (robot description, xacro)
@@ -42,4 +42,17 @@
     <mesh filename="${mesh}"/>
   </xacro:macro>
+  <!-- Use the per-link offset from the new visual config format when available,
+       otherwise retain the placement used by the old config format. -->
+  <xacro:macro name="mesh_origin" params="name legacy_xyz legacy_rpy">
+    <xacro:get_visual_params name="${name}" type="mesh_offset"/>
+    <xacro:if value="${visual_params != ''}">
+      <origin
+        xyz="${visual_params['x']} ${visual_params['y']} ${visual_params['z']}"
+        rpy="${visual_params['roll']} ${visual_params['pitch']} ${visual_params['yaw']}"/>
+    </xacro:if>
+    <xacro:unless value="${visual_params != ''}">
+      <origin xyz="${legacy_xyz}" rpy="${legacy_rpy}"/>
+    </xacro:unless>
+  </xacro:macro>
   <xacro:macro name="read_model_data" params="joint_limits_parameters_file kinematics_parameters_file physical_parameters_file visual_parameters_file force_abs_paths">
     <xacro:property name="force_abs_paths" value="${force_abs_paths}" scope="parent"/>
@@ -51,8 +64,9 @@
     <!-- Extract subsections from yaml dictionaries -->
     <xacro:property name="sec_limits" value="${config_joint_limit_parameters['joint_limits']}"/>
-    <xacro:property name="sec_offsets" value="${config_physical_parameters['offsets']}"/>
     <xacro:property name="sec_inertia_parameters" value="${config_physical_parameters['inertia_parameters']}" />
     <xacro:property name="sec_mesh_files" value="${config_visual_parameters['mesh_files']}" scope="parent"/>
     <xacro:property name="sec_kinematics" value="${config_kinematics_parameters['kinematics']}" />
+    <!-- Models that omit this key default to no Smart Panel. -->
+    <xacro:property name="smart_panel_from_visual" value="${config_visual_parameters['smart_panel'] if 'smart_panel' in config_visual_parameters else False}" scope="parent"/>
     <!-- JOINTS LIMIT PARAMETERS -->
     <xacro:property name="shoulder_pan_lower_limit" value="${sec_limits['shoulder_pan_joint']['min_position']}" scope="parent"/>
@@ -124,6 +138,6 @@
     <xacro:property name="wrist_3_yaw" value="${sec_kinematics['wrist_3']['yaw']}" scope="parent"/>
     <!-- OFFSETS -->
-    <xacro:property name="shoulder_offset" value="${sec_offsets['shoulder_offset']}" scope="parent"/>
-    <xacro:property name="elbow_offset" value="${sec_offsets['elbow_offset']}" scope="parent"/>
+    <xacro:property name="shoulder_offset" value="${config_physical_parameters['offsets']['shoulder_offset'] if 'offsets' in config_physical_parameters and 'shoulder_offset' in config_physical_parameters['offsets'] else 0.0}" scope="parent"/>
+    <xacro:property name="elbow_offset" value="${config_physical_parameters['offsets']['elbow_offset'] if 'offsets' in config_physical_parameters and 'elbow_offset' in config_physical_parameters['offsets'] else 0.0}" scope="parent"/>
     <!-- INERTIA PARAMETERS -->
     <!-- mass -->
@@ -208,10 +222,4 @@
     <xacro:property name="wrist_3_inertia_iyz" value="${prop_wrist_3_inertia['iyz']}" scope="parent"/>
     <xacro:property name="wrist_3_inertia_izz" value="${prop_wrist_3_inertia['izz']}" scope="parent"/>
-    <!-- cylinder radius -->
-    <xacro:property name="shoulder_radius" value="${sec_inertia_parameters['shoulder_radius']}" scope="parent"/>
-    <xacro:property name="upper_arm_radius" value="${sec_inertia_parameters['upper_arm_radius']}" scope="parent"/>
-    <xacro:property name="elbow_radius" value="${sec_inertia_parameters['elbow_radius']}" scope="parent"/>
-    <xacro:property name="forearm_radius" value="${sec_inertia_parameters['forearm_radius']}" scope="parent"/>
-    <xacro:property name="wrist_radius" value="${sec_inertia_parameters['wrist_radius']}" scope="parent"/>
     <!--KINEMATICS HASH-->
     <xacro:property name="kinematics_hash" value="${sec_kinematics['hash']}" scope="parent"/>

File: urdf/ur.urdf.xacro (robot description, xacro)
@@ -5,5 +5,5 @@
    <!-- import main macro -->
    <xacro:include filename="$(find ur_description)/urdf/ur_macro.xacro"/>
-   <!-- possible 'ur_type' values: ur3, ur5, ur10, ur3e, ur5e, ur7e, ur10e, ur12e, ur16e, ur8long, ur15, ur18, ur20, ur30 -->
+   <!-- possible 'ur_type' values: ur3, ur5, ur10, ur3e, ur5e, ur7e, ur10e, ur12e, ur16e, ur8long, ur15, ur18, ur20, ur30, ur10g-1750, ur17g-1300, ur18g-950 -->
    <!-- the default value should raise an error in case this was called without defining the type -->
    <xacro:arg name="ur_type" default="ur5x"/>
@@ -20,4 +20,6 @@
    <!--When using gazebo simulations absolute paths are necessary.-->
    <xacro:arg name="force_abs_paths" default="false" />
+   <!-- Empty default uses the value from visual_parameters.yaml (false if omitted). -->
+   <xacro:arg name="smart_panel" default="" />
    <!-- create link fixed to the "world" -->
    <link name="world" />
@@ -35,4 +37,5 @@
      safety_k_position="$(arg safety_k_position)"
      force_abs_paths="$(arg force_abs_paths)"
+     smart_panel="$(arg smart_panel)"
      >
      <origin xyz="0 0 0" rpy="0 0 0" />          <!-- position robot in the world -->

File: urdf/ur_macro.xacro (robot description, xacro)
@@ -56,4 +56,5 @@
     safety_k_position:=20
     force_abs_paths:=false
+    smart_panel:=''
     ">
     <!-- Load configuration data from the provided .yaml files -->
@@ -64,4 +65,6 @@
       visual_parameters_file="${visual_parameters_file}"
       force_abs_paths="${force_abs_paths}"/>
+    <!-- Empty smart_panel argument means "use visual_parameters.yaml". -->
+    <xacro:property name="smart_panel_enabled" value="${smart_panel if smart_panel != '' else smart_panel_from_visual}"/>
     <!-- links -  main serial chain -->
     <!-- base_link serves as the root of the robot's kinematic tree. It follows REP-103
@@ -74,5 +77,5 @@
     <link name="${tf_prefix}base_link_inertia">
       <visual>
-        <origin xyz="0 0 0" rpy="0 0 ${pi}"/>
+        <xacro:mesh_origin name="base" legacy_xyz="0 0 0" legacy_rpy="0 0 ${pi}"/>
         <geometry>
           <xacro:get_mesh name="base" type="visual"/>
@@ -80,5 +83,5 @@
       </visual>
       <collision>
-        <origin xyz="0 0 0" rpy="0 0 ${pi}"/>
+        <xacro:mesh_origin name="base" legacy_xyz="0 0 0" legacy_rpy="0 0 ${pi}"/>
         <geometry>
           <xacro:get_mesh name="base" type="collision"/>
@@ -91,5 +94,5 @@
     <link name="${tf_prefix}shoulder_link">
       <visual>
-        <origin xyz="0 0 0" rpy="0 0 ${pi}"/>
+        <xacro:mesh_origin name="shoulder" legacy_xyz="0 0 0" legacy_rpy="0 0 ${pi}"/>
         <geometry>
           <xacro:get_mesh name="shoulder" type="visual"/>
@@ -97,5 +100,5 @@
       </visual>
       <collision>
-        <origin xyz="0 0 0" rpy="0 0 ${pi}"/>
+        <xacro:mesh_origin name="shoulder" legacy_xyz="0 0 0" legacy_rpy="0 0 ${pi}"/>
         <geometry>
           <xacro:get_mesh name="shoulder" type="collision"/>
@@ -116,5 +119,5 @@
     <link name="${tf_prefix}upper_arm_link">
       <visual>
-        <origin xyz="0 0 ${shoulder_offset}" rpy="${pi/2} 0 ${-pi/2}"/>
+        <xacro:mesh_origin name="upper_arm" legacy_xyz="0 0 ${shoulder_offset}" legacy_rpy="${pi/2} 0 ${-pi/2}"/>
         <geometry>
           <xacro:get_mesh name="upper_arm" type="visual"/>
@@ -122,5 +125,5 @@
       </visual>
       <collision>
-        <origin xyz="0 0 ${shoulder_offset}" rpy="${pi/2} 0 ${-pi/2}"/>
+        <xacro:mesh_origin name="upper_arm" legacy_xyz="0 0 ${shoulder_offset}" legacy_rpy="${pi/2} 0 ${-pi/2}"/>
         <geometry>
           <xacro:get_mesh name="upper_arm" type="collision"/>
@@ -142,5 +145,5 @@
     <link name="${tf_prefix}forearm_link">
       <visual>
-        <origin xyz="0 0 ${elbow_offset}" rpy="${pi/2} 0 ${-pi/2}"/>
+        <xacro:mesh_origin name="forearm" legacy_xyz="0 0 ${elbow_offset}" legacy_rpy="${pi/2} 0 ${-pi/2}"/>
         <geometry>
           <xacro:get_mesh name="forearm" type="visual"/>
@@ -148,5 +151,5 @@
       </visual>
       <collision>
-        <origin xyz="0 0 ${elbow_offset}" rpy="${pi/2} 0 ${-pi/2}"/>
+        <xacro:mesh_origin name="forearm" legacy_xyz="0 0 ${elbow_offset}" legacy_rpy="${pi/2} 0 ${-pi/2}"/>
         <geometry>
           <xacro:get_mesh name="forearm" type="collision"/>
@@ -167,7 +170,8 @@
     </link>
     <link name="${tf_prefix}wrist_1_link">
-	  <xacro:get_visual_params name="wrist_1" type="visual_offset"/>
-      <visual>
-      	<origin xyz="0 0 ${visual_params}" rpy="${pi/2} 0 0"/>
+      <xacro:get_visual_params name="wrist_1" type="visual_offset"/>
+      <xacro:property name="wrist_1_legacy_offset" value="${visual_params}"/>
+      <visual>
+        <xacro:mesh_origin name="wrist_1" legacy_xyz="0 0 ${wrist_1_legacy_offset}" legacy_rpy="${pi/2} 0 0"/>
         <geometry>
           <xacro:get_mesh name="wrist_1" type="visual"/>
@@ -175,5 +179,5 @@
       </visual>
       <collision>
-        <origin xyz="0 0 ${visual_params}" rpy="${pi/2} 0 0"/>
+        <xacro:mesh_origin name="wrist_1" legacy_xyz="0 0 ${wrist_1_legacy_offset}" legacy_rpy="${pi/2} 0 0"/>
         <geometry>
           <xacro:get_mesh name="wrist_1" type="collision"/>
@@ -194,7 +198,8 @@
     </link>
     <link name="${tf_prefix}wrist_2_link">
-          <xacro:get_visual_params name="wrist_2" type="visual_offset"/>
-      <visual>
-        <origin xyz="0 0 ${visual_params}" rpy="0 0 0"/>
+      <xacro:get_visual_params name="wrist_2" type="visual_offset"/>
+      <xacro:property name="wrist_2_legacy_offset" value="${visual_params}"/>
+      <visual>
+        <xacro:mesh_origin name="wrist_2" legacy_xyz="0 0 ${wrist_2_legacy_offset}" legacy_rpy="0 0 0"/>
         <geometry>
           <xacro:get_mesh name="wrist_2" type="visual"/>
@@ -202,5 +207,5 @@
       </visual>
       <collision>
-        <origin xyz="0 0 ${visual_params}" rpy="0 0 0"/>
+        <xacro:mesh_origin name="wrist_2" legacy_xyz="0 0 ${wrist_2_legacy_offset}" legacy_rpy="0 0 0"/>
         <geometry>
           <xacro:get_mesh name="wrist_2" type="collision"/>
@@ -229,5 +234,5 @@
       </xacro:if>
       <visual>
-        <origin xyz="${mesh_offset}" rpy="${pi/2} 0 0"/>
+        <xacro:mesh_origin name="wrist_3" legacy_xyz="${mesh_offset}" legacy_rpy="${pi/2} 0 0"/>
         <geometry>
           <xacro:get_mesh name="wrist_3" type="visual"/>
@@ -235,5 +240,5 @@
       </visual>
       <collision>
-        <origin xyz="${mesh_offset}" rpy="${pi/2} 0 0"/>
+        <xacro:mesh_origin name="wrist_3" legacy_xyz="${mesh_offset}" legacy_rpy="${pi/2} 0 0"/>
         <geometry>
           <xacro:get_mesh name="wrist_3" type="collision"/>
@@ -375,4 +380,45 @@
       <origin xyz="0 0 0" rpy="0 ${-pi/2.0} ${-pi/2.0}" />
     </joint>
+    <!-- Optional Smart Panel accessory attached to wrist_3_link.
+         Geometry lives in meshes/common/smart_panel so it can be reused
+         across robot models. -->
+    <xacro:if value="${smart_panel_enabled}">
+      <xacro:if value="${force_abs_paths}">
+        <xacro:property name="smart_panel_visual_mesh" value="file://$(find ur_description)/meshes/common/smart_panel/visual/smart_panel.dae"/>
+        <xacro:property name="smart_panel_collision_mesh" value="file://$(find ur_description)/meshes/common/smart_panel/collision/smart_panel.stl"/>
+      </xacro:if>
+      <xacro:unless value="${force_abs_paths}">
+        <xacro:property name="smart_panel_visual_mesh" value="package://ur_description/meshes/common/smart_panel/visual/smart_panel.dae"/>
+        <xacro:property name="smart_panel_collision_mesh" value="package://ur_description/meshes/common/smart_panel/collision/smart_panel.stl"/>
+      </xacro:unless>
+      <link name="${tf_prefix}smart_panel">
+        <visual>
+          <origin xyz="0 0 0" rpy="0 0 0"/>
+          <geometry>
+            <mesh filename="${smart_panel_visual_mesh}"/>
+          </geometry>
+        </visual>
+        <collision>
+          <origin xyz="0 0 0" rpy="0 0 0"/>
+          <geometry>
+            <mesh filename="${smart_panel_collision_mesh}"/>
+          </geometry>
+        </collision>
+        <inertial>
+          <!-- Inertia estimated for homogeneous weight distribution and the measured mass of the smart panel. -->
+          <origin xyz="0.045 0 -0.030" rpy="0 0 0"/>
+          <mass value="0.0195"/>
+          <inertia ixx="5.682064e-06" ixy="4.66603e-10" ixz="1.863097e-07"
+                   iyy="3.330845e-06" iyz="-2.165772e-09"
+                   izz="3.256972e-06"/>
+        </inertial>
+      </link>
+      <joint name="${tf_prefix}wrist_3_link-smart_panel" type="fixed">
+        <parent link="${tf_prefix}wrist_3_link"/>
+        <child link="${tf_prefix}smart_panel"/>
+        <!-- the mesh is in the correct position relative to wrist_3_link -->
+        <origin xyz="0 0 0" rpy="0 0 0"/>
+      </joint>
+    </xacro:if>
     <!-- ROS-Industrial 'tool0' frame - all-zeros tool frame -->
     <link name="${tf_prefix}tool0"/>

File: urdf/ur_mocked.urdf.xacro (robot description, xacro)
@@ -6,5 +6,5 @@
   <xacro:include filename="$(find ur_description)/urdf/ur_macro.xacro"/>
   <xacro:include filename="$(find ur_description)/urdf/ros2_control_mock_hardware.xacro" />
-  <!-- possible 'ur_type' values: ur3, ur5, ur10, ur3e, ur5e, ur7e, ur10e, ur12e, ur16e, ur8long, ur15, ur18, ur20, ur30 -->
+  <!-- possible 'ur_type' values: ur3, ur5, ur10, ur3e, ur5e, ur7e, ur10e, ur12e, ur16e, ur8long, ur15, ur18, ur20, ur30, ur10g-1750, ur17g-1300, ur18g-950 -->
   <!-- the default value should raise an error in case this was called without defining the type -->
   <xacro:arg name="ur_type" default="ur5x"/>
@@ -22,4 +22,6 @@
   <!--When using gazebo simulations absolute paths are necessary.-->
   <xacro:arg name="force_abs_paths" default="false" />
+  <!-- Empty default uses the value from visual_parameters.yaml (false if omitted). -->
+  <xacro:arg name="smart_panel" default="" />
   <!-- initial position for simulations (Mock Hardware, Gazebo, Ignition) -->
   <xacro:arg name="initial_positions_file" default="$(find ur_description)/config/initial_positions.yaml"/>
@@ -41,4 +43,5 @@
     safety_k_position="$(arg safety_k_position)"
     force_abs_paths="$(arg force_abs_paths)"
+    smart_panel="$(arg smart_panel)"
     >
     <origin xyz="0 0 0" rpy="0 0 0" />          <!-- position robot in the world -->
