Commit message: Imported upstream version '4.4.0' of 'upstream'

File: urdf/inc/ur_common.xacro (robot description, xacro)
@@ -41,17 +41,4 @@
     <xacro:get_mesh_path/>
     <mesh filename="${mesh}"/>
-  </xacro:macro>
-  <!-- Use the per-link offset from the new visual config format when available,
-       otherwise retain the placement used by the old config format. -->
-  <xacro:macro name="mesh_origin" params="name legacy_xyz legacy_rpy">
-    <xacro:get_visual_params name="${name}" type="mesh_offset"/>
-    <xacro:if value="${visual_params != ''}">
-      <origin
-        xyz="${visual_params['x']} ${visual_params['y']} ${visual_params['z']}"
-        rpy="${visual_params['roll']} ${visual_params['pitch']} ${visual_params['yaw']}"/>
-    </xacro:if>
-    <xacro:unless value="${visual_params != ''}">
-      <origin xyz="${legacy_xyz}" rpy="${legacy_rpy}"/>
-    </xacro:unless>
   </xacro:macro>
   <xacro:macro name="read_model_data" params="joint_limits_parameters_file kinematics_parameters_file physical_parameters_file visual_parameters_file force_abs_paths">
@@ -137,7 +124,4 @@
     <xacro:property name="wrist_3_pitch" value="${sec_kinematics['wrist_3']['pitch']}" scope="parent"/>
     <xacro:property name="wrist_3_yaw" value="${sec_kinematics['wrist_3']['yaw']}" scope="parent"/>
-    <!-- OFFSETS -->
-    <xacro:property name="shoulder_offset" value="${config_physical_parameters['offsets']['shoulder_offset'] if 'offsets' in config_physical_parameters and 'shoulder_offset' in config_physical_parameters['offsets'] else 0.0}" scope="parent"/>
-    <xacro:property name="elbow_offset" value="${config_physical_parameters['offsets']['elbow_offset'] if 'offsets' in config_physical_parameters and 'elbow_offset' in config_physical_parameters['offsets'] else 0.0}" scope="parent"/>
     <!-- INERTIA PARAMETERS -->
     <!-- mass -->

File: urdf/ur_macro.xacro (robot description, xacro)
@@ -76,6 +76,9 @@
     <link name="${tf_prefix}base_link"/>
     <link name="${tf_prefix}base_link_inertia">
-      <visual>
-        <xacro:mesh_origin name="base" legacy_xyz="0 0 0" legacy_rpy="0 0 ${pi}"/>
+      <xacro:get_visual_params name="base" type="mesh_offset"/>
+      <visual>
+        <origin
+         xyz="${visual_params['x']} ${visual_params['y']} ${visual_params['z']}"
+         rpy="${visual_params['roll']} ${visual_params['pitch']} ${visual_params['yaw']}"/>
         <geometry>
           <xacro:get_mesh name="base" type="visual"/>
@@ -83,5 +86,7 @@
       </visual>
       <collision>
-        <xacro:mesh_origin name="base" legacy_xyz="0 0 0" legacy_rpy="0 0 ${pi}"/>
+        <origin
+         xyz="${visual_params['x']} ${visual_params['y']} ${visual_params['z']}"
+         rpy="${visual_params['roll']} ${visual_params['pitch']} ${visual_params['yaw']}"/>
         <geometry>
           <xacro:get_mesh name="base" type="collision"/>
@@ -93,6 +98,9 @@
     </link>
     <link name="${tf_prefix}shoulder_link">
-      <visual>
-        <xacro:mesh_origin name="shoulder" legacy_xyz="0 0 0" legacy_rpy="0 0 ${pi}"/>
+      <xacro:get_visual_params name="shoulder" type="mesh_offset"/>
+      <visual>
+        <origin
+         xyz="${visual_params['x']} ${visual_params['y']} ${visual_params['z']}"
+         rpy="${visual_params['roll']} ${visual_params['pitch']} ${visual_params['yaw']}"/>
         <geometry>
           <xacro:get_mesh name="shoulder" type="visual"/>
@@ -100,5 +108,7 @@
       </visual>
       <collision>
-        <xacro:mesh_origin name="shoulder" legacy_xyz="0 0 0" legacy_rpy="0 0 ${pi}"/>
+        <origin
+         xyz="${visual_params['x']} ${visual_params['y']} ${visual_params['z']}"
+         rpy="${visual_params['roll']} ${visual_params['pitch']} ${visual_params['yaw']}"/>
         <geometry>
           <xacro:get_mesh name="shoulder" type="collision"/>
@@ -118,6 +128,9 @@
       </inertial>    </link>
     <link name="${tf_prefix}upper_arm_link">
-      <visual>
-        <xacro:mesh_origin name="upper_arm" legacy_xyz="0 0 ${shoulder_offset}" legacy_rpy="${pi/2} 0 ${-pi/2}"/>
+      <xacro:get_visual_params name="upper_arm" type="mesh_offset"/>
+      <visual>
+        <origin
+         xyz="${visual_params['x']} ${visual_params['y']} ${visual_params['z']}"
+         rpy="${visual_params['roll']} ${visual_params['pitch']} ${visual_params['yaw']}"/>
         <geometry>
           <xacro:get_mesh name="upper_arm" type="visual"/>
@@ -125,5 +138,7 @@
       </visual>
       <collision>
-        <xacro:mesh_origin name="upper_arm" legacy_xyz="0 0 ${shoulder_offset}" legacy_rpy="${pi/2} 0 ${-pi/2}"/>
+        <origin
+         xyz="${visual_params['x']} ${visual_params['y']} ${visual_params['z']}"
+         rpy="${visual_params['roll']} ${visual_params['pitch']} ${visual_params['yaw']}"/>
         <geometry>
           <xacro:get_mesh name="upper_arm" type="collision"/>
@@ -144,6 +159,9 @@
     </link>
     <link name="${tf_prefix}forearm_link">
-      <visual>
-        <xacro:mesh_origin name="forearm" legacy_xyz="0 0 ${elbow_offset}" legacy_rpy="${pi/2} 0 ${-pi/2}"/>
+      <xacro:get_visual_params name="forearm" type="mesh_offset"/>
+      <visual>
+        <origin
+         xyz="${visual_params['x']} ${visual_params['y']} ${visual_params['z']}"
+         rpy="${visual_params['roll']} ${visual_params['pitch']} ${visual_params['yaw']}"/>
         <geometry>
           <xacro:get_mesh name="forearm" type="visual"/>
@@ -151,5 +169,7 @@
       </visual>
       <collision>
-        <xacro:mesh_origin name="forearm" legacy_xyz="0 0 ${elbow_offset}" legacy_rpy="${pi/2} 0 ${-pi/2}"/>
+        <origin
+         xyz="${visual_params['x']} ${visual_params['y']} ${visual_params['z']}"
+         rpy="${visual_params['roll']} ${visual_params['pitch']} ${visual_params['yaw']}"/>
         <geometry>
           <xacro:get_mesh name="forearm" type="collision"/>
@@ -170,8 +190,9 @@
     </link>
     <link name="${tf_prefix}wrist_1_link">
-      <xacro:get_visual_params name="wrist_1" type="visual_offset"/>
-      <xacro:property name="wrist_1_legacy_offset" value="${visual_params}"/>
-      <visual>
-        <xacro:mesh_origin name="wrist_1" legacy_xyz="0 0 ${wrist_1_legacy_offset}" legacy_rpy="${pi/2} 0 0"/>
+      <xacro:get_visual_params name="wrist_1" type="mesh_offset"/>
+      <visual>
+        <origin
+         xyz="${visual_params['x']} ${visual_params['y']} ${visual_params['z']}"
+         rpy="${visual_params['roll']} ${visual_params['pitch']} ${visual_params['yaw']}"/>
         <geometry>
           <xacro:get_mesh name="wrist_1" type="visual"/>
@@ -179,5 +200,7 @@
       </visual>
       <collision>
-        <xacro:mesh_origin name="wrist_1" legacy_xyz="0 0 ${wrist_1_legacy_offset}" legacy_rpy="${pi/2} 0 0"/>
+        <origin
+         xyz="${visual_params['x']} ${visual_params['y']} ${visual_params['z']}"
+         rpy="${visual_params['roll']} ${visual_params['pitch']} ${visual_params['yaw']}"/>
         <geometry>
           <xacro:get_mesh name="wrist_1" type="collision"/>
@@ -198,8 +221,9 @@
     </link>
     <link name="${tf_prefix}wrist_2_link">
-      <xacro:get_visual_params name="wrist_2" type="visual_offset"/>
-      <xacro:property name="wrist_2_legacy_offset" value="${visual_params}"/>
-      <visual>
-        <xacro:mesh_origin name="wrist_2" legacy_xyz="0 0 ${wrist_2_legacy_offset}" legacy_rpy="0 0 0"/>
+      <xacro:get_visual_params name="wrist_2" type="mesh_offset"/>
+      <visual>
+        <origin
+         xyz="${visual_params['x']} ${visual_params['y']} ${visual_params['z']}"
+         rpy="${visual_params['roll']} ${visual_params['pitch']} ${visual_params['yaw']}"/>
         <geometry>
           <xacro:get_mesh name="wrist_2" type="visual"/>
@@ -207,5 +231,7 @@
       </visual>
       <collision>
-        <xacro:mesh_origin name="wrist_2" legacy_xyz="0 0 ${wrist_2_legacy_offset}" legacy_rpy="0 0 0"/>
+        <origin
+         xyz="${visual_params['x']} ${visual_params['y']} ${visual_params['z']}"
+         rpy="${visual_params['roll']} ${visual_params['pitch']} ${visual_params['yaw']}"/>
         <geometry>
           <xacro:get_mesh name="wrist_2" type="collision"/>
@@ -226,13 +252,9 @@
     </link>
     <link name="${tf_prefix}wrist_3_link">
-      <!-- TODO: remove this once all wrist_3 meshes have the visual_offset_xyz tag -->
-      <xacro:get_visual_params name="wrist_3" type="visual_offset_xyz"/>
-      <xacro:property name="mesh_offset" value="${visual_params}" scope="parent"/>
-      <xacro:if value="${visual_params == ''}">
-        <xacro:get_visual_params name="wrist_3" type="visual_offset"/>
-        <xacro:property name="mesh_offset" value="0 0 ${visual_params}" scope="parent"/>
-      </xacro:if>
-      <visual>
-        <xacro:mesh_origin name="wrist_3" legacy_xyz="${mesh_offset}" legacy_rpy="${pi/2} 0 0"/>
+      <xacro:get_visual_params name="wrist_3" type="mesh_offset"/>
+      <visual>
+        <origin
+         xyz="${visual_params['x']} ${visual_params['y']} ${visual_params['z']}"
+         rpy="${visual_params['roll']} ${visual_params['pitch']} ${visual_params['yaw']}"/>
         <geometry>
           <xacro:get_mesh name="wrist_3" type="visual"/>
@@ -240,5 +262,7 @@
       </visual>
       <collision>
-        <xacro:mesh_origin name="wrist_3" legacy_xyz="${mesh_offset}" legacy_rpy="${pi/2} 0 0"/>
+        <origin
+         xyz="${visual_params['x']} ${visual_params['y']} ${visual_params['z']}"
+         rpy="${visual_params['roll']} ${visual_params['pitch']} ${visual_params['yaw']}"/>
         <geometry>
           <xacro:get_mesh name="wrist_3" type="collision"/>

Commit message: Rebase from 'upstream'

File: urdf/inc/ur_common.xacro (robot description, xacro)
@@ -54,4 +54,6 @@
     <xacro:property name="sec_mesh_files" value="${config_visual_parameters['mesh_files']}" scope="parent"/>
     <xacro:property name="sec_kinematics" value="${config_kinematics_parameters['kinematics']}" />
+    <!-- Models that omit this key default to no Smart Panel. -->
+    <xacro:property name="smart_panel_from_visual" value="${config_visual_parameters['smart_panel'] if 'smart_panel' in config_visual_parameters else False}" scope="parent"/>
     <!-- JOINTS LIMIT PARAMETERS -->
     <xacro:property name="shoulder_pan_lower_limit" value="${sec_limits['shoulder_pan_joint']['min_position']}" scope="parent"/>

File: urdf/ur_macro.xacro (robot description, xacro)
@@ -56,4 +56,5 @@
     safety_k_position:=20
     force_abs_paths:=false
+    smart_panel:=''
     ">
     <!-- Load configuration data from the provided .yaml files -->
@@ -64,4 +65,6 @@
       visual_parameters_file="${visual_parameters_file}"
       force_abs_paths="${force_abs_paths}"/>
+    <!-- Empty smart_panel argument means "use visual_parameters.yaml". -->
+    <xacro:property name="smart_panel_enabled" value="${smart_panel if smart_panel != '' else smart_panel_from_visual}"/>
     <!-- links -  main serial chain -->
     <!-- base_link serves as the root of the robot's kinematic tree. It follows REP-103
@@ -401,4 +404,45 @@
       <origin xyz="0 0 0" rpy="0 ${-pi/2.0} ${-pi/2.0}" />
     </joint>
+    <!-- Optional Smart Panel accessory attached to wrist_3_link.
+         Geometry lives in meshes/common/smart_panel so it can be reused
+         across robot models. -->
+    <xacro:if value="${smart_panel_enabled}">
+      <xacro:if value="${force_abs_paths}">
+        <xacro:property name="smart_panel_visual_mesh" value="file://$(find ur_description)/meshes/common/smart_panel/visual/smart_panel.dae"/>
+        <xacro:property name="smart_panel_collision_mesh" value="file://$(find ur_description)/meshes/common/smart_panel/collision/smart_panel.stl"/>
+      </xacro:if>
+      <xacro:unless value="${force_abs_paths}">
+        <xacro:property name="smart_panel_visual_mesh" value="package://ur_description/meshes/common/smart_panel/visual/smart_panel.dae"/>
+        <xacro:property name="smart_panel_collision_mesh" value="package://ur_description/meshes/common/smart_panel/collision/smart_panel.stl"/>
+      </xacro:unless>
+      <link name="${tf_prefix}smart_panel">
+        <visual>
+          <origin xyz="0 0 0" rpy="0 0 0"/>
+          <geometry>
+            <mesh filename="${smart_panel_visual_mesh}"/>
+          </geometry>
+        </visual>
+        <collision>
+          <origin xyz="0 0 0" rpy="0 0 0"/>
+          <geometry>
+            <mesh filename="${smart_panel_collision_mesh}"/>
+          </geometry>
+        </collision>
+        <inertial>
+          <!-- Inertia estimated for homogeneous weight distribution and the measured mass of the smart panel. -->
+          <origin xyz="0.045 0 -0.030" rpy="0 0 0"/>
+          <mass value="0.0195"/>
+          <inertia ixx="5.682064e-06" ixy="4.66603e-10" ixz="1.863097e-07"
+                   iyy="3.330845e-06" iyz="-2.165772e-09"
+                   izz="3.256972e-06"/>
+        </inertial>
+      </link>
+      <joint name="${tf_prefix}wrist_3_link-smart_panel" type="fixed">
+        <parent link="${tf_prefix}wrist_3_link"/>
+        <child link="${tf_prefix}smart_panel"/>
+        <!-- the mesh is in the correct position relative to wrist_3_link -->
+        <origin xyz="0 0 0" rpy="0 0 0"/>
+      </joint>
+    </xacro:if>
     <!-- ROS-Industrial 'tool0' frame - all-zeros tool frame -->
     <link name="${tf_prefix}tool0"/>
